File: Adafruit Metro RP2350.kicad_pcb (KiCad board)
At the start: 4 copper layers, 55 x 65.6 mm, 64 parts, among them J1 USB_C_Receptacle_USB2.0_14P, J2 Conn_02x09_Counter_Clockwise, J3 Conn_01x05_Pin, SW2 SW_RA, SW3 SW_RA, U1 APS1604M-3SQRx-SN, U2 W25Q128JVS, U4 74LVC1G19, U5 NCP1117-3.3_SOT223, U7 APS1604M-3SQRx-SN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

Commit message: prot1
Parts:
- moved J2 19.0 mm to (59.8, 119.3), turned to 180 degrees
Connections:
- J2 pad 10: /D23 -> /D8
- J2 pad 11: /D1 -> /D7
- J2 pad 12: /D3 -> /D6
- J2 pad 14: /D7 -> /D4
- J2 pad 15: /D8 -> /D3
- J2 pad 16: /D9 -> /D2
- J2 pad 17: /SDA -> /RT
- J2 pad 18: GND -> /PD
- J2 pad 2: /SCL -> GND
- J2 pad 3: /D10 -> /SCL
- J2 pad 4: /D11 -> /SDA
- J2 pad 5: /D6 -> /VS
- J2 pad 6: /D4 -> /HS
- J2 pad 7: /D2 -> /PC
- J2 pad 8: /D0 -> /XC
- J2 pad 9: /D22 -> /D9
- R11 pad 1: /D23 -> /PD
- X4 pad 1: /D4 -> /D7
- X4 pad 2: /D5 -> /D6
- X4 pad 22: /D22 -> /RT
- X4 pad 23: /D23 -> /PD
- X4 pad 3: /D6 -> /D9
- X4 pad 4: /D7 -> /D8
- X4 pad 6: /D8 -> /XC
- X4 pad 7: /D9 -> /HS
- X4 pad 77: /D0 -> /D3
- X4 pad 78: /D1 -> /D2
- X4 pad 79: /D2 -> /D5
- X4 pad 8: /D10 -> /VS
- X4 pad 80: /D3 -> /D4
- X4 pad 9: /D11 -> /PC
Routing:
- net /PD: track 0.00 -> 95.9 mm, vias 0 -> 2
- net /RT: track 0.00 -> 53.4 mm, vias 0 -> 3
- net /D1: track 52.3 -> 0.00 mm, vias 2 -> 0
- net /D10: track 46.8 -> 0.00 mm, vias 5 -> 0
- net /VS: track 0.00 -> 44.3 mm, vias 0 -> 6
- net /D23: track 41.4 -> 0.00 mm, vias 5 -> 0
- net /D22: track 34.5 -> 0.00 mm, vias 2 -> 0
- net /XC: track 0.00 -> 31.2 mm, vias 0 -> 1
- net /D11: track 26.3 -> 0.00 mm, vias 3 -> 0
- net /D8: track 46.1 -> 19.9 mm, vias 8 -> 2
- net /D0: track 25.6 -> 0.00 mm, vias 3 -> 0
- net /D5: track 42.0 -> 64.2 mm, vias 5 -> 4
- net /HS: track 0.00 -> 21.2 mm, vias 0 -> 1
- net /PC: track 0.00 -> 18.7 mm, vias 0 -> 3
- net /SCL: track 46.0 -> 27.3 mm
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