File: hardware/proto2/kicad/Adafruit Metro RP2350.kicad_sch (KiCad schematic)
At the start: 107 parts, among them J1 USB_C_Receptacle_USB2.0_14P, J2 Conn_02x09_Counter_Clockwise, J3 Conn_01x05_Pin, U1 APS1604M-3SQRx-SN, U2 W25Q128JVS, U3 MCP2515-xST, U4 74LVC1G19, U5 NCP1117-3.3_SOT223, U6 SN65HVD230, U7 APS1604M-3SQRx-SN, U8 TLV74328, U9 TLV74315, X1 CAMERA_OV2640, X4 RP2350B, Y1 12MHz_10pF_50ohm

Commit message: proto2: smaller footprints, direct camera wiring, CAN block, 40x40 placement
- Passives moved to 0402 (10 uF to 0603), diodes to SOD-523, LEDs to 0402,
  with LCSC numbers for JLC basic/preferred parts where available
- All footprints from the standard KiCad libraries; Eagle-imported LED,
  diode, inductor and test point pins renumbered to match the pads
- Camera header pair (J2, JP1, JP2) removed and the camera wired straight
  to the RP2350B; D2-D9 now on GPIO0-7 in order; camera reset on its own
  net (GPIO22) instead of the RP2350 RUN net
- CAN: JST SH connector (J4), jumper-selectable 120 R terminator, MCP2515
  on SPI0 (GPIO32-35), INT on GPIO36, transceiver standby on GPIO37,
  16 MHz crystal
- A0 (GPIO41) no longer shorted to the MCP2515 3.3 V node
- SJ1 bridged to the RP2350 XCLK by default, OSC1 not populated
- Camera breakout power LED (D2, SJ3, R2) removed, ON0 populated
- PCB: 40 x 40 mm outline, old routing cleared, rough two-sided placement

Co-Authored-By: Claude Opus 5.5 <noreply@anthropic.com>
Parts:
- removed D2: GREEN, Adafruit OV5640 Breakout:CHIPLED_0603_NOOUTLINE, symbol Adafruit OV5640 Breakout-eagle-import:LED0603_NOOUTLINE
- removed J2: Conn_02x09_Counter_Clockwise, Connector_IDC:IDC-Header_2x09_P2.54mm_Vertical, symbol Connector_Generic:Conn_02x09_Counter_Clockwise
- removed JP1: HEADER-1X970MIL, Adafruit OV5640 Breakout:1X09_ROUND_70, symbol Adafruit OV5640 Breakout-eagle-import:HEADER-1X970MIL
- removed JP2: PINHD-2X9-BIG, Adafruit OV5640 Breakout:2X09-BIG, symbol Adafruit OV5640 Breakout-eagle-import:PINHD-2X9-BIG
- removed R2: 10K, Adafruit OV5640 Breakout:0603-NO, symbol Adafruit OV5640 Breakout-eagle-import:RESISTOR_0603_NOOUT
- removed SJ3: SOLDERJUMPERCLOSED, Adafruit OV5640 Breakout:SOLDERJUMPER_CLOSEDWIRE, symbol Adafruit OV5640 Breakout-eagle-import:SOLDERJUMPERCLOSED
- added C45: 100n, Capacitor_SMD:C_0402_1005Metric, symbol Device:C
- added C46, C47: 12pF, Capacitor_SMD:C_0402_1005Metric, symbol Device:C
- added J4: CAN, Connector_JST:JST_SH_SM03B-SRSS-TB_1x03-1MP_P1.00mm_Horizontal, symbol Connector_Generic_MountingPin:Conn_01x03_MountingPin
- added JP3: CAN_TERM, Jumper:SolderJumper-2_P1.3mm_Open_RoundedPad1.0x1.5mm, symbol Jumper:SolderJumper_2_Open
- added R31: 120, Resistor_SMD:R_0402_1005Metric, symbol Device:R
- added R32: 10K, Resistor_SMD:R_0402_1005Metric, symbol Device:R
- added Y2: 16MHz, Crystal:Crystal_SMD_3225-4Pin_3.2x2.5mm, symbol Device:Crystal_GND24
- C1, C4: footprint Capacitor_SMD:C_0603_1608Metric -> Capacitor_SMD:C_0402_1005Metric; LCSC C23630 -> C12530
- C10, C3, C34, C35: footprint Capacitor_SMD:C_0805_2012Metric -> Capacitor_SMD:C_0603_1608Metric; LCSC C15850 -> C96446
- C11, C12, C13, C16, C18, C2, C7, C9: footprint Capacitor_SMD:C_0603_1608Metric -> Capacitor_SMD:C_0402_1005Metric; LCSC C15849 -> C52923
- C14, C17, C20, C21, C22, C23, C24, C25, C33, C5, C6, C8: footprint Capacitor_SMD:C_0603_1608Metric -> Capacitor_SMD:C_0402_1005Metric; LCSC C14663 -> C1525
- C19: footprint Capacitor_SMD:C_0805_2012Metric -> Capacitor_SMD:C_0603_1608Metric; LCSC C6119932 -> C96446
- C26, C27: footprint Capacitor_SMD:C_0603_1608Metric -> Capacitor_SMD:C_0402_1005Metric; LCSC C1648 -> C1554
- C28: footprint Capacitor_SMD:C_0603_1608Metric -> Capacitor_SMD:C_0402_1005Metric; LCSC (none) -> C1525
- C29, C30, C31, C32, C36, C42, C43: footprint Adafruit OV5640 Breakout:0805-NO -> Capacitor_SMD:C_0603_1608Metric; LCSC (none) -> C96446
- C37, C38, C39, C40: footprint Adafruit OV5640 Breakout:0603-NO -> Capacitor_SMD:C_0402_1005Metric; LCSC (none) -> C1525
- C41: footprint Adafruit OV5640 Breakout:0603-NO -> Capacitor_SMD:C_0402_1005Metric; LCSC (none) -> C52923
- C44: footprint Adafruit OV5640 Breakout:0603-NO -> Capacitor_SMD:C_0402_1005Metric; LCSC (none) -> C1555
- D1: value 1N4148WS -> 1N4148WT; footprint Diode_SMD:D_SOD-323 -> Diode_SMD:D_SOD-523; LCSC (none) -> C7420320
- D3: footprint Diode_SMD:D_SOD-123 -> Diode_SMD:D_SOD-523; LCSC C81598 -> C7420320
- FB1: footprint Adafruit OV5640 Breakout:0603-NO -> Inductor_SMD:L_0402_1005Metric; LCSC (none) -> C76886
- L0, L2: footprint LED_SMD:LED_0603_1608Metric -> LED_SMD:LED_0402_1005Metric; LCSC C84256 -> C25503345
- L3: footprint LED_SMD:LED_0603_1608Metric -> LED_SMD:LED_0402_1005Metric; LCSC C84256 -> C965793
- L4: footprint LED_SMD:LED_0603_1608Metric -> LED_SMD:LED_0402_1005Metric; LCSC C84256 -> C25503856
- L5: footprint LED_SMD:LED_0603_1608Metric -> LED_SMD:LED_0402_1005Metric; LCSC C84256 -> C22355736
- L6: footprint LED_SMD:LED_0603_1608Metric -> LED_SMD:LED_0402_1005Metric; LCSC C19171390 -> C25503345
- ON0: footprint LED_SMD:LED_0603_1608Metric -> LED_SMD:LED_0402_1005Metric; LCSC C84256 -> C965793; now fitted
- OSC1: footprint Adafruit OV5640 Breakout:OSC_3.2X2.5MM -> Oscillator:Oscillator_SMD_Abracon_ASE-4Pin_3.2x2.5mm; LCSC (none) -> C712738; now not fitted
- R1, R3: footprint Resistor_SMD:R_0805_2012Metric -> Resistor_SMD:R_0402_1005Metric; LCSC C27834 -> C25905
- R10, R11, R12, R13: footprint Adafruit OV5640 Breakout:0603-NO -> Resistor_SMD:R_0402_1005Metric; LCSC (none) -> C25744
- R15: footprint Resistor_SMD:R_0805_2012Metric -> Resistor_SMD:R_0402_1005Metric; LCSC C228697 -> C25879
- R16, R21, R6, R9: footprint Resistor_SMD:R_0805_2012Metric -> Resistor_SMD:R_0402_1005Metric; LCSC C17414 -> C25744
- R17: footprint Resistor_SMD:R_0805_2012Metric -> Resistor_SMD:R_0402_1005Metric; LCSC C140868 -> C25744
- R23, R24, R25, R26, R27, R28, R29, R30: footprint Resistor_SMD:R_0805_2012Metric -> Resistor_SMD:R_0402_1005Metric; LCSC C17513 -> C11702
- R4: footprint Resistor_SMD:R_0805_2012Metric -> Resistor_SMD:R_0402_1005Metric; LCSC C17540 -> C25087
- R5: footprint Resistor_SMD:R_0805_2012Metric -> Resistor_SMD:R_0402_1005Metric; LCSC C17415 -> C25077
- R7, R8: footprint Resistor_SMD:R_0805_2012Metric -> Resistor_SMD:R_0402_1005Metric; LCSC C17561 -> C25092
- S1, S2: footprint lib_foot:SW_TS-1088-AR02016 -> Button_Switch_SMD:SW_SPST_TS-1088-xR020
- SJ1: footprint Adafruit OV5640 Breakout:SOLDERJUMPER_2WAY_OPEN_NOPASTE -> Jumper:SolderJumper-3_P1.3mm_Bridged12_RoundedPad1.0x1.5mm_NumberLabels
- SJ2: footprint Adafruit OV5640 Breakout:SOLDERJUMPER_ARROW_NOPASTE -> Jumper:SolderJumper-2_P1.3mm_Open_RoundedPad1.0x1.5mm
- TP2: footprint Adafruit OV5640 Breakout:TESTPOINT_ROUND_1.5MM -> TestPoint:TestPoint_Pad_D1.5mm
- U8: footprint Adafruit OV5640 Breakout:SOT23-5 -> Package_TO_SOT_SMD:SOT-23-5; LCSC (none) -> C408971
- U9: footprint Adafruit OV5640 Breakout:SOT23-5 -> Package_TO_SOT_SMD:SOT-23-5; LCSC (none) -> C469895
- X1: footprint Adafruit OV5640 Breakout:OV2640FSL -> Connector_FFC-FPC:Jushuo_AFC07-S24FCA-00_1x24-1MP_P0.50_Horizontal; LCSC (none) -> C262567
Connections:
- net D2 is gone; now on net DATA3: X4.78 (CS0/RX0/SCL0/PWM0B/GPIO1)
- net D3 is gone; now on net DATA2: X4.77 (XPI_CS1/MISO0/TX0/SDA0/PWM0A/GPIO0)
- net D4 is gone; now on net DATA5: X4.80 (MOSI0/RTS0/SCL1/PWM1B/GPIO3)
- net D5 is gone; now on net DATA4: X4.79 (SCK0/CTS0/SDA1/PWM1A/GPIO2)
- net D6 is gone; now on net DATA7: X4.2 (CS0/RX1/SCL0/PWM2B/GPIO5)
- net D7 is gone; now on net DATA6: X4.1 (MISO0/TX1/SDA0/PWM2A/GPIO4)
- net D8 is gone; now on net DATA9: X4.4 (MOSI0/RTS1/SCL1/PWM3B/GPIO7)
- net D9 is gone; now on net DATA8: X4.3 (SCK0/CTS1/SDA1/PWM3A/GPIO6)
- net HS is gone; now on net HSYNC: X4.7 (CS1/RX1/SCL0/PWM4B/GPIO9)
- net PC is gone; now on net PCLK: X4.9 (MOSI1/RTS1/SCL1/PWM5B/GPIO11)
- net PD is gone; now on net PWDN: R30.2, X4.23 (MOSI0/RTS1/SCL1/PWM3B/GPIO23)
- net VS is gone; now on net VSYNC: X4.8 (SCK1/CTS1/SDA1/PWM5A/GPIO10)
- net XC is gone; now on net EXT_XCLK: X4.6 (XIP_CS1/MISO1/TX1/SDA0/PWM4A/GPIO8)
- net 1.2V: now also L1.1; no longer L1.P$1 (1)
- net 3.3V: now also U6.3 (VCC), C45.1; no longer R15.1, R24.2, X4.52 (GPIO41/ADC1/CS1/TX1/SCL0/PWM8B)
- net GND: now also L0.1 (C), L2.1 (C), L3.1 (C), L4.1 (C), L5.1 (C), L6.1 (C), ON0.1 (C), U6.2 (GND), X1.MP (DGND), C45.2, C46.2, C47.2, J4.3 (Pin_3), J4.MP (MountPin), R32.2, Y2.2 (G), Y2.4 (G); no longer L0.C, L2.C, L3.C, L4.C, L5.C, L6.C, ON0.C, X1.SPRT1 (DGND), X1.SPRT2 (DGND)
- net LX: now also L1.2; no longer L1.P$2 (2)
- net STROBE: now also TP2.1 (P$1); no longer TP2.P$1
- net USBBOOT: now also D3.1 (C), TP1.1 (P$1); no longer D3.C, TP1.P$1
- net ~{RESET}: no longer C40.1, R10.2, X1.6 (~{RESET})
- net at R26.2: now also D3.2 (A); no longer D3.A
- net at R29.1: now also ON0.2 (A); no longer ON0.A
- net CAN_TX: now reaches U3.1 (TXCAN)
- net CAN_TX: now also U6.1 (D)
- net CAN_INT: now reaches U3.13 (~{INT})
- net CAN_INT: now also X4.45 (GPIO36/MISO0/TX1/SDA0/PWM10A)
- net CAN_SCK: now reaches U3.14 (SCK)
- net CAN_SCK: now also X4.43 (GPIO34/SCK0/CTS0/SDA1/PWM9A)
- net CAN_MOSI: now reaches U3.16 (SI)
- net CAN_MOSI: now also X4.44 (GPIO35/MOSI0/RTS0/SCL1/PWM9B)
- net CAN_MISO: now reaches U3.17 (SO)
- net CAN_MISO: now also X4.40 (GPIO32/MISO0/TX0/SDA0/PWM8A)
- net CAN_CS: now reaches U3.18 (~{CS})
- net CAN_CS: now also X4.42 (GPIO33/CS0/RX0/SCL0/PWM8B)
- net CAN_RX: now reaches U3.2 (RXCAN)
- net CAN_RX: now also U6.4 (R)
- net CAN_OSC2: now reaches U3.8 (OSC2)
- net CAN_OSC2: now also C47.1, Y2.3
- net CAN_OSC1: now reaches U3.9 (OSC1)
- net CAN_OSC1: now also C46.1, Y2.1
- net at R30.1: now also L0.2 (A); no longer L0.A
- net at R15.2: now also L6.2 (A); no longer L6.A
- net at R24.1: now also L2.2 (A); no longer L2.A
- net at R25.1: now also L3.2 (A); no longer L3.A
- net CANL: now reaches U6.6 (CANL)
- net CANL: now also J4.2 (Pin_2), R31.2
- net CANH: now reaches U6.7 (CANH)
- net CANH: now also J4.1 (Pin_1), JP3.1 (A)
- net CAN_STBY: now reaches U6.8 (Rs)
- net CAN_STBY: now also X4.46 (GPIO37/CS0/RX1/SCL0/PWM10B), R32.1
- net at R28.1: now also L5.2 (A); no longer L5.A
- net at R27.1: now also L4.2 (A); no longer L4.A
- net RT renamed CAM_~{RESET}
- net CAM_~{RESET}: now also C40.1, R10.2, X1.6 (~{RESET})
- new net: JP3.2 (B), R31.1
- new net A0: R15.1, R24.2, X4.52 (GPIO41/ADC1/CS1/TX1/SCL0/PWM8B)
- no-connect marks 0 -> 7
Other:
- note removed: "ON LED"
